Commit message: Faster training with faster simulation

File: sim/assets/robots/turtlebot/turtlebot.urdf (robot description, URDF)
Before this commit: robot turtlebot, 34 links, 33 joints
Links:
- link wheel_left_link: geometry collision cylinder length=0.0206 radius=0.0650; visual mesh filename=turtlebot/kobuki_description/meshes/wheel.dae
- link wheel_right_link: geometry collision cylinder length=0.0206 radius=0.0650; visual mesh filename=turtlebot/kobuki_description/meshes/wheel.dae
Joints:
- joint wheel_left_joint: origin xyz=0.00 0.115 0.0250 rpy=-1.57079632679 0 0 -> xyz=0.00 0.115 0.0550 rpy=-1.57079632679 0 0
- joint wheel_right_joint: origin xyz=0.00 -0.115 0.0250 rpy=-1.57079632679 0 0 -> xyz=0.00 -0.115 0.0550 rpy=-1.57079632679 0 0
